Commit message: thunder computer and mppi

File: src/rm_bnrobot_sim/urdf/bngu_sentinel/actuator/wheel.urdf.xacro (robot description, xacro)
@@ -19,5 +19,5 @@
                 </geometry>
             </collision>
-            <xacro:cylinder_inertia m="0.1" h="0.04" r="0.055"/>
+            <xacro:cylinder_inertia m="0.6" h="0.04" r="0.055"/>
         </link>
         <!-- Gazebo物理参数 -->

File: src/rm_bnrobot_sim/urdf/bngu_sentinel/base.urdf.xacro (robot description, xacro)
@@ -2,24 +2,7 @@
 <robot xmlns:xacro="http://www.ros.org/wiki/xacro">
     <xacro:include filename="$(find rm_bnrobot_sim)/urdf/bngu_sentinel/common_inertia.xacro" />
-    <!-- 关键修改：参数从 length radius → length width height（长、宽、高独立可控） -->
     <xacro:macro name="base_xacro" params="length width height">
-        <link name="base_footprint" />
-        <joint name="base_joint" type="fixed">
-            <parent link="base_footprint" />
-            <child link="base_link" />
-            <origin xyz="0.0 0.0 ${height/2.0+0.055-0.008}" rpy="0 0 0" />
-        </joint>
         <link name="base_link">
             <visual>
-                <origin xyz="0 0 0.0" rpy="0 0 0" />
-                <geometry>
-                    <box size="${length} ${width} ${height}" /> <!-- 长×宽×高 -->
-                </geometry>
-                <material name="blue">
-                    <color rgba="0.1 0.1 1.0 0.5"/>
-                </material>
-            </visual>
-            <!-- 碰撞：与视觉尺寸一致 -->
-            <collision>
                 <origin xyz="0 0 0.0" rpy="0 0 0" />
                 <geometry>
@@ -29,4 +12,10 @@
                     <color rgba="0.1 0.1 1.0 0.5"/>
                 </material>
+            </visual>
+            <collision>
+                <origin xyz="0 0 0.0" rpy="0 0 0" />
+                <geometry>
+                    <box size="${length} ${width} ${height}" />
+                </geometry>
             </collision>
             <xacro:box_inertia m="1.0" w="${length}" h="${width}" d="${height}"/>

File: src/rm_bnrobot_sim/urdf/bngu_sentinel/bnbot.urdf.xacro (robot description, xacro)
@@ -14,19 +14,17 @@
     <!-- 传感器 -->
     <xacro:laser_xacro xyz="0 0 0.105" />
-    <!-- 1. Mid360: 相对于base_link的位姿 (extrinsic_T + extrinsic_R) -->
-    <xacro:mid360 name="mid360_laser" topic="/mid360/pointcloud">
+    <xacro:mid360 name="mid360_laser" topic="/livox/lidar">
         <origin xyz="0 0 0.6" rpy="${M_PI} 0 ${M_PI/2}" />
     </xacro:mid360>
-    <!-- 2. IMU: 挂载到mid360_laser_link (而非base_link)，使用相对位姿 -->
-    <joint name="imu_to_mid360_joint" type="fixed">
-        <parent link="mid360_laser_link" />  <!-- Mid360的link名称，需和mid360.urdf.xacro一致 -->
-        <child link="imu_link" />             <!-- IMU的link名称，需和imu.urdf.xacro一致 -->
-        <origin xyz="-0.011 -0.02329 0.04412" rpy="0 0 0" />  <!-- IMU相对于Mid360的位姿 -->
+    <!-- <joint name="imu_to_mid360_joint" type="fixed">
+        <parent link="mid360_laser" />
+        <child link="imu_link" />
+        <origin xyz="-0.011 -0.02329 0.04412" rpy="0 0 0" />
         <axis xyz="0 0 0" />
-    </joint>
+    </joint> -->
+    <xacro:imu_xacro xyz="0 0 0.6" />
     <!-- <xacro:imu_xacro xyz="0 0 0.02" /> -->
     <!-- <xacro:imu_xacro xyz="0 0 0.02" /> -->
-    <!-- <xacro:imu_xacro xyz="0 0 0.02" /> -->
-    <!-- <xacro:camera_xacro xyz="0.10 0 0.45" /> -->
+    <xacro:camera_xacro xyz="0.10 0 0.45" />
     <!-- <xacro:mid360 name="mid360_laser" topic="/mid360/pointcloud"> <origin xyz="0.2665 0.0 0.145" rpy="0 0 0" /></xacro:mid360> -->
     <!-- 麦克纳姆轮配置，保持原有轮距参数 -->
@@ -37,5 +35,5 @@
     <!-- Gazebo 插件 -->
     <xacro:include filename="$(find rm_bnrobot_sim)/urdf/bngu_sentinel/plugins/gazebo_control_plugin.xacro" />
-    <xacro:gazebo_control_plugin /> <!-- 启用平面运动插件 -->
+    <xacro:gazebo_control_plugin />
     <xacro:include filename="$(find rm_bnrobot_sim)/urdf/bngu_sentinel/bnbot.ros2_control.xacro" />
     <xacro:bngu_sentinel_ros2_control />

File: src/rm_bnrobot_sim/urdf/bngu_sentinel/bnbot_real.xacro (robot description, xacro)
@@ -1,24 +1,17 @@
 <?xml version="1.0" encoding="UTF-8"?>
 <robot name="bnbot" xmlns:xacro="http://ros.org/wiki/xacro" ns="bnbot">
-  <!-- 1. 提取可配置参数（后续修改直接改这里，无需动结构） -->
-  <xacro:property name="M_PI" value="3.1415926" />  <!-- 通用常量 -->
-  <!-- 底座参数 -->
-  <xacro:property name="base_length" value="0.633" />  <!-- 长(x) -->
-  <xacro:property name="base_width" value="0.526" />   <!-- 宽(y) -->
-  <xacro:property name="base_height" value="0.42" />   <!-- 高(z) -->
-  <xacro:property name="base_mass" value="5.0" />      <!-- 质量(kg) -->
-  <xacro:property name="base_center_z" value="${base_height/2}" />  <!-- 底座中心z坐标（自动计算，避免硬编码） -->
-  <!-- 雷达安装参数 -->
-  <xacro:property name="lidar_install_z" value="${base_height}" />  <!-- 雷达安装在底座上表面（z=底座总高度） -->
-  <xacro:property name="lidar_topic" value="mid360" />  <!-- 雷达发布话题（与之前配置一致） -->
-  <!-- 2. 地面参考帧（不变） -->
-  <link name="base_footprint" />
-  <!-- 3. 核心底座（使用参数化配置） -->
+  <xacro:property name="M_PI" value="3.1415926" />
+  <xacro:property name="base_length" value="0.633" />
+  <xacro:property name="base_width" value="0.526" />
+  <xacro:property name="base_height" value="0.42" />
+  <xacro:property name="base_mass" value="5.0" />
+  <xacro:property name="base_center_z" value="${base_height/2}" /> <xacro:property name="lidar_topic" value="mid360" />
+  <xacro:include filename="$(find ros2_livox_simulation)/urdf/mid360.xacro" />
+  <link name="mid360" />
   <link name="base_link">
     <visual>
-      <!-- 用参数替代硬编码，中心z坐标自动计算 -->
       <origin xyz="0 0 ${base_center_z}" rpy="0 0 0" />
       <geometry>
-        <box size="${base_length} ${base_width} ${base_height}" />  <!-- 参数化尺寸 -->
+        <box size="${base_length} ${base_width} ${base_height}" />
       </geometry>
       <material name="blue">
@@ -26,5 +19,4 @@
       </material>
     </visual>
-    <!-- 碰撞体与视觉体一致（参数化） -->
     <collision>
       <origin xyz="0 0 ${base_center_z}" rpy="0 0 0" />
@@ -33,23 +25,18 @@
       </geometry>
     </collision>
-    <!-- 惯性参数（参数化质量） -->
     <inertial>
-      <mass value="${base_mass}" />  <!-- 用参数替代硬编码 -->
+      <origin xyz="0 0 ${base_center_z}" rpy="0 0 0" />
+      <mass value="${base_mass}" />
       <inertia ixx="0.01" ixy="0.0" ixz="0.0"
-               iyy="0.01" iyz="0.0" izz="0.02" /> <!-- 简化惯性矩阵，可根据实际优化 -->
+               iyy="0.01" iyz="0.0" izz="0.02" />
     </inertial>
   </link>
-  <!-- 4. base_footprint到base_link的固定关节（参数化z轴高度） -->
-  <joint name="base_joint" type="fixed">
-    <parent link="base_footprint" />
+  <joint name="mid360_to_base_joint" type="fixed">
+    <parent link="mid360" />
     <child link="base_link" />
-    <origin xyz="0.0 0.0 ${base_center_z}" rpy="0 0 0" />  <!-- z=底座中心高度（下表面贴地） -->
+    <origin xyz="0 0 -${base_height+0.2}" rpy="0 0 0" />
   </joint>
-  <!-- 5. 集成Livox Mid360激光雷达（保持原有宏调用，参数化配置） -->
-  <!-- 包含Mid360的xacro文件（确保ros2_livox_simulation功能包已编译安装） -->
-  <xacro:include filename="$(find ros2_livox_simulation)/urdf/mid360.xacro" />
-  <!-- 调用Mid360宏：使用参数化安装位置和话题 -->
-  <xacro:mid360 name="mid360" parent="base_link" topic="${lidar_topic}" >
-    <origin xyz="0 0 ${lidar_install_z}" rpy="0 0 0"/>
+  <xacro:mid360 name="mid360_sensor" parent="mid360" topic="${lidar_topic}">
+    <origin xyz="0 0 0" rpy="0 0 0"/>
   </xacro:mid360>
 </robot>

File: src/rm_bnrobot_sim/urdf/bngu_sentinel/plugins/gazebo_control_plugin.xacro (robot description, xacro)
@@ -25,7 +25,7 @@
                 <!-- 输出配置 -->
                 <publish_odom>true</publish_odom>
-                <publish_odom_tf>false</publish_odom_tf>
+                <publish_odom_tf>true</publish_odom_tf>
                 <odometry_frame>odom</odometry_frame>
-                <robot_base_frame>base_footprint</robot_base_frame>
+                <robot_base_frame>base_link</robot_base_frame>
             </plugin>
         </gazebo>

File: src/rm_bnrobot_sim/urdf/bngu_sentinel/plugins/gazebo_sensor_plugin.xacro (robot description, xacro)
@@ -46,9 +46,10 @@
     <sensor name="imu_sensor" type="imu">
         <plugin name="imu_plugin" filename="libgazebo_ros_imu_sensor.so">
+            <frame_name>imu_link</frame_name>
             <ros>
                 <namespace>/</namespace>
-                <remapping>~/out:=imu</remapping>
+                <remapping>~/out:=livox/imu</remapping>
             </ros>
-            <initial_orientation_as_reference>false</initial_orientation_as_reference>
+            <initial_orientation_as_reference>true</initial_orientation_as_reference>
         </plugin>
         <update_rate>100</update_rate>

File: src/rm_bnrobot_sim/urdf/bngu_sentinel/sensor/imu.urdf.xacro (robot description, xacro)
@@ -5,5 +5,5 @@
         <link name="imu_link">
             <visual>
-                <origin xyz="0 0 00" rpy="0 0 0" />
+                <origin xyz="0 0 0" rpy="0 0 0" />
                 <geometry>
                     <box size="0.02 0.02 0.02" />
@@ -27,5 +27,5 @@
             <parent link="base_link" />
             <child link="imu_link" />
-            <origin xyz="${xyz}" />
+            <origin xyz="${xyz}" rpy="${M_PI} 0 ${M_PI/2}" />
         </joint>
     </xacro:macro>

File: src/rm_bnrobot_sim/urdf/bngu_sentinel/sensor/mid360.urdf.xacro (robot description, xacro)
@@ -22,5 +22,5 @@
   <xacro:property name="downsample_rate" value="2" /> <!-- 降采样系数（2=每2个点保留1个） -->
   <!-- 2. 雷达模型-->
-  <xacro:macro name="mid360" params=" name:='mid360_laser' parent:='base_link' topic:='/mid360/pointcloud' *origin">
+  <xacro:macro name="mid360" params=" name:='mid360_laser' parent:='base_link' topic:='/livox/lidar' *origin">
     <link name="${name}">
       <visual>
@@ -28,5 +28,5 @@
         <origin xyz="0.025 -0.0265 -0.025" rpy="${M_PI/2} 0 ${M_PI}"/>
         <geometry>
-          <mesh filename="file:///home/mage/navigation/nav_RM_4/src/rm_bnrobot_sim/meshes/mid360.stl" scale="0.0008 0.0008 0.0008"/>
+          <mesh filename="file:///home/nav2/navigation_2027/navi_rm_0/src/rm_bnrobot_sim/meshes/mid360.stl" scale="0.0008 0.0008 0.0008"/>
         </geometry>
         <material name="black">
@@ -92,5 +92,5 @@
             </noise>
           </ray>
-          <visualize>false</visualize> <!-- 点云可视化由RViz负责，Gazebo中关闭 -->
+          <visualize>true</visualize> <!-- 点云可视化由RViz负责，Gazebo中关闭 -->
           <samples>${horizontal_samples * vertical_samples}</samples> <!-- 总采样数 -->
           <downsample>${downsample_rate}</downsample> <!-- 降采样 -->
